Commit message: update

File: espresso_frame_gazebo_launch/urdf/all.urdf (robot description, URDF)
Before this commit: robot test_robot, 5 links, 4 joints
Links:
- added link frame_link
- added link top_camera_link
Joints:
- added joint frame_joint: type fixed, parent base_link, child frame_link, origin xyz=-0.140 0 0.052 rpy=0 0 0
- added joint top_camera_joint: type fixed, parent frame_link, child top_camera_link, origin xyz=0.014 0 0.990 rpy=0 0 0
- joint front_laser_joint: origin xyz=0.140 0 0 rpy=0 0 3.141592 -> xyz=0.140 0 0.010 rpy=0 0 3.141592
- joint head_camera_joint: origin xyz=0.03 0 0 rpy=0 0 0 -> xyz=0.044 0 0 rpy=0 0 0
- joint turret_base_joint: origin xyz=0 0 0.6 rpy=0 0 0 -> xyz=0.095 0 0.673 rpy=0 0 0; parent base_link -> frame_link
